Commit message: changed some frames

File: urdf/base.xacro (robot description, xacro)
@@ -10,5 +10,5 @@
         <visual>
             <geometry>
-                <mesh filename="file://$(find hey_agv_new)/urdf/agv_base.dae"/>
+                <mesh filename="file://$(find master_server)/urdf/agv_base.dae"/>
             </geometry>
             <origin xyz="0 0 0" rpy="0 0 1.5708" />
@@ -18,5 +18,5 @@
         <collision>
             <geometry>
-                <mesh filename="file://$(find hey_agv_new)/urdf/agv_base.dae"/>
+                <mesh filename="file://$(find master_server)/urdf/agv_base.dae"/>
             </geometry>
              <origin xyz="0 0 0" rpy="0 0 1.5708" />
@@ -60,5 +60,5 @@
         <axis xyz="0 1 0" />
     </joint>
-    <link name="${robot_prefix}lidar_right">
+    <link name="${robot_prefix}lidar_right_link">
         <visual>
             <geometry>
@@ -77,8 +77,8 @@
     <joint name="${robot_prefix}lidar_right_base_joint" type="fixed">
         <parent link="${robot_prefix}base_link" />
-        <child link="${robot_prefix}lidar_right" />
-        <origin xyz="0.115 -0.16789 0.12" rpy="0 0 0"/>
-    </joint>
-    <link name="${robot_prefix}lidar_left">
+        <child link="${robot_prefix}lidar_right_link" />
+        <origin xyz="0.115 -0.16789 0.12" rpy="0 0 3.14"/>
+    </joint>
+    <link name="${robot_prefix}lidar_left_link">
         <visual>
             <geometry>
@@ -97,6 +97,6 @@
     <joint name="${robot_prefix}lidar_left_base_joint" type="fixed">
         <parent link="${robot_prefix}base_link" />
-        <child link="${robot_prefix}lidar_left" />
-        <origin xyz="-0.115 0.16789 0.12" rpy="0 0 3.14"/>
+        <child link="${robot_prefix}lidar_left_link" />
+        <origin xyz="-0.115 0.16789 0.12" rpy="0 0 0"/>
     </joint>
     <!-- make a square lift -->
